File: front/core.kicad_sch (KiCad schematic)
At the start: 1 part, among them U2 TCA9548APWR

Commit message: start adding components
Parts:
- removed U2: TCA9548APWR, Package_SO:TSSOP-24_4.4x7.8mm_P0.65mm, symbol Interface_Expansion:TCA9548APWR
- added U5: TCA9548APWR, Package_SO:TSSOP-24_4.4x7.8mm_P0.65mm, symbol Interface_Expansion:TCA9548APWR
Changed lines of the file:
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@@
 	(symbol
 		(lib_id "Interface_Expansion:TCA9548APWR")
-		(at 140.97 74.93 0)
+		(at 147.32 96.52 0)
 		(unit 1)
 		(exclude_from_sim no)
@@
 		(dnp no)
 		(fields_autoplaced yes)
-		(property "Reference" "U2"
-			(at 143.1133 49.53 0)
+		(property "Reference" "U5"
+			(at 149.4633 71.12 0)
 			(effects
 				(font
@@
 		)
 		(property "Value" "TCA9548APWR"
-			(at 143.1133 52.07 0)
+			(at 149.4633 73.66 0)
 			(effects
 				(font
@@
 		)
 		(property "Footprint" "Package_SO:TSSOP-24_4.4x7.8mm_P0.65mm"
-			(at 140.97 100.33 0)
+			(at 147.32 121.92 0)
 			(effects
 				(font
@@
 		)
 		(property "Datasheet" "http://www.ti.com/lit/ds/symlink/tca9548a.pdf"
-			(at 142.24 68.58 0)
+			(at 148.59 90.17 0)
 			(effects
 				(font
@@
 		)
 		(property "Description" "Low voltage 8-channel I2C switch with reset, TSSOP-24"
-			(at 140.97 74.93 0)
+			(at 147.32 96.52 0)
 			(effects
 				(font
@@
 			)
 		)
-		(pin "18"
+		(pin "3"
 		)
 		(pin "22"
 		)
+		(pin "23"
+		)
+		(pin "21"
+		)
+		(pin "2"
+		)
 		(pin "1"
 		)
-		(pin "23"
+		(pin "24"
+		)
+		(pin "18"
+		)
+		(pin "6"
+		)
+		(pin "14"
+		)
+		(pin "17"
+		)
+		(pin "16"
+		)
+		(pin "13"
+		)
+		(pin "20"
 		)
 		(pin "5"
 		)
-		(pin "24"
+		(pin "9"
 		)
-		(pin "9"
+		(pin "19"
+		)
+		(pin "11"
+		)
+		(pin "12"
+		)
+		(pin "4"
+		)
+		(pin "15"
+		)
+		(pin "10"
 		)
 		(pin "8"
 		)
-		(pin "21"
-		)
-		(pin "4"
-		)
-		(pin "10"
-		)
-		(pin "13"
-		)
-		(pin "15"
-		)
-		(pin "6"
-		)
-		(pin "11"
-		)
-		(pin "20"
-		)
-		(pin "14"
-		)
-		(pin "12"
-		)
-		(pin "19"
-		)
 		(pin "7"
-		)
-		(pin "2"
-		)
-		(pin "3"
-		)
-		(pin "16"
-		)
-		(pin "17"
 		)
 		(instances
 			(project ""
-				(path "/81e90ab1-1e02-4123-b0b3-bb0377a29c19"
-					(reference "U2")
+				(path "/508f986b-6f1b-4c39-bd57-bae69573a4e7/d0e6b8f3-b2a8-43c8-8076-7747d5419a72"
+					(reference "U5")
 					(unit 1)
 				)
@@
 		)
 	)
-	(sheet_instances
-		(path "/"
-			(page "1")
-		)
-	)
-	(embedded_fonts no)
 )
