File: front/front.kicad_pcb (KiCad board)
At the start: 2 copper layers, 18.4 x 17.1 mm, 1 part, among them U1 VL53L8CXV0GC/1

Commit message: start adding components
Parts:
- added U2: VL53L8CXV0GC/1, Library:IC17_LGA16_STM, F.Cu at (77.7, 105.6)
- added U3: TCA9548APWR, Package_SO:TSSOP-24_4.4x7.8mm_P0.65mm, F.Cu at (77.5, 161.3)
- added U4: PCA9615DP, Package_SO:TSSOP-10_3x3mm_P0.5mm, F.Cu at (201.9, 87.6)
- U1: value VL53L8CXV0GC/1 -> LSM6DSO32TR; footprint Library:IC17_LGA16_STM -> Library:XDCR_LSM6DSO32TR
- moved U1 54.7 mm to (76.2, 41.9)
Other:
- board size 18.4 x 17.1 mm -> 182.2 x 132.1 mm
