File: front/front.kicad_pcb (KiCad board)
At the start: 2 copper layers, 189.2 x 82.2 mm, 8 parts, among them J1 Conn_01x04, J2 Conn_01x04, J3 Conn_01x04, U1 LSM6DSO32TR, U2 VL53L8CXV0GC/1, U3 TCA9548APWR, U4 PCA9615DP

Commit message: add more components
Parts:
- added C2: 100n, Capacitor_SMD:C_0603_1608Metric, F.Cu at (83.4, 116.6)
- added C3: 100n, Capacitor_SMD:C_0603_1608Metric, F.Cu at (78.7, 109.2)
- added C4: 4.7u, Capacitor_SMD:C_0603_1608Metric, F.Cu at (78.0, 101.3)
- added C5: 100n, Capacitor_SMD:C_0603_1608Metric, F.Cu at (87.6, 39.2)
- added C6: 100n, Capacitor_SMD:C_0603_1608Metric, F.Cu at (87.6, 41.7)
- added C7: 100n, Capacitor_SMD:C_0603_1608Metric, F.Cu at (87.6, 44.2)
- added C8: 10u, Capacitor_SMD:C_0603_1608Metric, F.Cu at (81.9, 113.5)
- added C9: 1u, Capacitor_SMD:C_0603_1608Metric, F.Cu at (76.0, 112.5)
- added J4: Conn_01x04_Pin, Connector_PinHeader_2.54mm:PinHeader_1x04_P2.54mm_Horizontal, B.Cu at (82.0, 97.1)
- added NT1: NetTie_3, Jumper:SolderJumper-3_P1.3mm_Bridged12_RoundedPad1.0x1.5mm, F.Cu at (66.0, 40.6)
- added R1: 47k, Resistor_SMD:R_0603_1608Metric, F.Cu at (73.3, 114.3)
- added R2: 47k, Resistor_SMD:R_0603_1608Metric, F.Cu at (73.3, 116.9)
- added R3: 47k, Resistor_SMD:R_0603_1608Metric, F.Cu at (80.3, 101.3)
- added R4: 47k, Resistor_SMD:R_0603_1608Metric, F.Cu at (83.1, 107.4)
- added R5: 47k, Resistor_SMD:R_0603_1608Metric, F.Cu at (83.1, 103.9)
- added R6: R, Resistor_SMD:R_0603_1608Metric, F.Cu at (72.9, 111.0)
- added R7: R, Resistor_SMD:R_0603_1608Metric, F.Cu at (74.2, 101.3)
- added U5: LDK130M18R, Library:SOT23-5L_1P75X3P05X0P95_STM, F.Cu at (79.0, 115.3)
- C1: value 1uF -> 100n
- U3: value TCA9548APWR -> PCA9848PWJ; footprint Package_SO:TSSOP-24_4.4x7.8mm_P0.65mm -> Library:TSSOP24_SOT355-1_NEX_NXP
- moved C1 10.6 mm to (67.6, 37.1), turned to 180 degrees
- moved U1 2.30 mm to (82.8, 41.1)
- moved U3 0.80 mm to (72.1, 41.9), turned to 90 degrees
Connections:
- C1 pad 1: Net-(U3-VCC) -> /top/1.8v
- U1 pad 1: unconnected-(U1-SDO/SA0-Pad1) -> GND
- U1 pad 12: unconnected-(U1-CS-Pad12) -> /top/1.8v
- U1 pad 13: unconnected-(U1-SCL-Pad13) -> /top/scimu
- U1 pad 14: unconnected-(U1-SDA-Pad14) -> /top/sdimu
- U1 pad 2: unconnected-(U1-SDX-Pad2) -> GND
- U1 pad 3: unconnected-(U1-SCX-Pad3) -> GND
- U1 pad 5: unconnected-(U1-VDDIO-Pad5) -> /top/1.8v
- U1 pad 8: unconnected-(U1-VDD-Pad8) -> /top/1.8v
- U2 pad A1: unconnected-(U2-INT-PadA1) -> Net-(U2-INT)
- U2 pad A2: unconnected-(U2-LPN-PadA2) -> Net-(U2-LPN)
- U2 pad A3: unconnected-(U2-IOVDD-PadA3) -> /sensorC/1.8v
- U2 pad A4: unconnected-(U2-SDA/MOSI-PadA4) -> /sensorC/sd_vl
- U2 pad A5: unconnected-(U2-SCL/MCLK-PadA5) -> /sensorC/sc_vl
- U2 pad A6: unconnected-(U2-RSVD1-PadA6) -> GND
- U2 pad A7: unconnected-(U2-RSVD2-PadA7) -> GND
- U2 pad B1: unconnected-(U2-SYNC-PadB1) -> Net-(U2-SYNC)
- U2 pad B7: unconnected-(U2-CORE_1V8-PadB7) -> /sensorC/1.8v
- U2 pad C1: unconnected-(U2-SPI_I2C_N-PadC1) -> Net-(U2-SPI_I2C_N)
- U2 pad C2: unconnected-(U2-NCS-PadC2) -> Net-(U2-NCS)
- U2 pad C3: unconnected-(U2-GND-PadC3) -> GND
- U2 pad C4: unconnected-(U2-AVDD-PadC4) -> /sensorC/3.3v
- U2 pad C6: unconnected-(U2-RSVD3-PadC6) -> GND
- U2 pad C7: unconnected-(U2-GROUND-PadC7) -> GND
- U3 pad 1: unconnected-(U3-A0-Pad1) -> /top/1.8v
- U3 pad 10: unconnected-(U3-SD3-Pad10) -> /top/sd3
- U3 pad 11: unconnected-(U3-SC3-Pad11) -> /top/sc3
- U3 pad 13: unconnected-(U3-SD4-Pad13) -> /top/sdimu
- U3 pad 14: unconnected-(U3-SC4-Pad14) -> /top/scimu
- U3 pad 2: unconnected-(U3-A1-Pad2) -> /top/1.8v
- U3 pad 21: unconnected-(U3-A2-Pad21) -> Net-(U3-A1)
- U3 pad 22: unconnected-(U3-SCL-Pad22) -> /top/scl
- U3 pad 23: unconnected-(U3-SDA-Pad23) -> /top/sda
- U3 pad 24: Net-(U3-VCC) -> /top/1.8v
- U3 pad 3: unconnected-(U3-~{RESET}-Pad3) -> /top/1.8v
- U3 pad 6: unconnected-(U3-SD1-Pad6) -> /top/sd1
- U3 pad 7: unconnected-(U3-SC1-Pad7) -> /top/sc1
- U3 pad 8: unconnected-(U3-SD2-Pad8) -> /top/sd2
- U3 pad 9: unconnected-(U3-SC2-Pad9) -> /top/sc2
Routing:
- net /top/1.8v: track 0.00 -> 8.21 mm
- net unconnected-(U2-SDA/MOSI-PadA4): track 2.69 -> 0.00 mm

Commit message: begin layout
Parts:
- added C10: 100n, Capacitor_SMD:C_0603_1608Metric, F.Cu at (230.9, 96.0)
- added C11: 1u, Capacitor_SMD:C_0603_1608Metric, F.Cu at (230.9, 98.5)
- added C12: 10n, Capacitor_SMD:C_0402_1005Metric, F.Cu at (200.9, 85.4)
- added C13: 4.7u, Capacitor_SMD:C_0603_1608Metric, F.Cu at (210.0, 93.5)
- added C14: 22u, Capacitor_SMD:C_0805_2012Metric, F.Cu at (210.4, 99.6)
- added J5: Conn_01x06_Pin, Connector_PinSocket_2.54mm:PinSocket_1x06_P2.54mm_Vertical, F.Cu at (79.8, 37.3)
- added J6: Conn_01x06_Pin, Connector_PinHeader_2.54mm:PinHeader_1x06_P2.54mm_Horizontal, B.Cu at (216.2, 82.8)
- added L1: 2.2u, Inductor_SMD:L_Vishay_IHLP-3232, F.Cu at (195.3, 98.0)
- added L2: 1u, Library:INDC2520X120N, F.Cu at (215.1, 94.0)
- added NT0: NetTie_3, Jumper:SolderJumper-3_P1.3mm_Bridged12_RoundedPad1.0x1.5mm, F.Cu at (67.3, 48.0)
- added NT3: NetTie_3, Jumper:SolderJumper-3_P1.3mm_Bridged12_RoundedPad1.0x1.5mm, F.Cu at (236.7, 86.9)
- added R10: 200k, Resistor_SMD:R_0603_1608Metric, F.Cu at (206.2, 91.2)
- added R11: 100k, Resistor_SMD:R_0603_1608Metric, F.Cu at (206.2, 93.7)
- added R8: 61.9k, Resistor_SMD:R_0603_1608Metric, F.Cu at (194.8, 91.9)
- added R9: 249k, Resistor_SMD:R_0603_1608Metric, F.Cu at (194.8, 89.4)
- added REF**: MountingHole_2.2mm_M2_DIN965, MountingHole:MountingHole_2.2mm_M2_DIN965, F.Cu at (77.5, 111.5)
- added U6: TLV62568ADRL, Package_TO_SOT_SMD:SOT-563, F.Cu at (205.9, 96.6)
- C8: footprint Capacitor_SMD:C_0603_1608Metric -> Capacitor_SMD:C_0805_2012Metric
- C9: value 1u -> 22u; footprint Capacitor_SMD:C_0603_1608Metric -> Capacitor_SMD:C_0805_2012Metric
- J1, J2, J3: value Conn_01x04 -> Conn_01x05; footprint Connector_PinHeader_2.54mm:PinHeader_1x04_P2.54mm_Vertical -> Connector_PinHeader_2.54mm:PinHeader_1x05_P2.54mm_Vertical
- J4: value Conn_01x04_Pin -> Conn_01x05_Pin; footprint Connector_PinHeader_2.54mm:PinHeader_1x04_P2.54mm_Horizontal -> Connector_PinHeader_2.54mm:PinHeader_1x05_P2.54mm_Horizontal
- U5: value LDK130M18R -> TPS62902RPJR; footprint Library:SOT23-5L_1P75X3P05X0P95_STM -> Library:IC_TPS62902RPJR
- moved U1 154.5 mm to (231.3, 83.8)
- moved C6 154.4 mm to (236.5, 82.6)
- moved C7 149.3 mm to (230.6, 87.1)
- moved C9 123.6 mm to (195.8, 82.1), turned to 180 degrees
- moved C8 117.5 mm to (195.8, 85.1), turned to 180 degrees
- moved U5 117.4 mm to (191.2, 80.8), turned to 180 degrees
- moved U4 36.9 mm to (237.2, 98.3)
- moved C5 17.9 mm to (71.4, 46.7)
- moved R2 15.3 mm to (71.9, 101.6)
- moved R6 12.3 mm to (79.5, 100.6)
- moved R5 11.2 mm to (71.9, 104.6), turned to 180 degrees
- moved C2 11.0 mm to (82.5, 105.7), turned to 90 degrees
- moved R3 10.5 mm to (71.9, 107.7), turned to 0 degrees
- moved R4 9.94 mm to (74.7, 102.1)
- moved C4 8.85 mm to (81.5, 109.4), turned to 0 degrees
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Connections:
- C6 pad 1: /top/1.8v -> /back/3.3v
- C7 pad 1: /top/1.8v -> /back/3.3v
- C8 pad 1: /sensorC/1.8v -> /back/bat+
- C9 pad 1: /sensorC/3.3v -> /back/3.3v
- J1 pad 1: unconnected-(J1-Pin_1-Pad1) -> GND
- J1 pad 2: unconnected-(J1-Pin_2-Pad2) -> /top/3.3v
- J1 pad 3: unconnected-(J1-Pin_3-Pad3) -> /top/sc_vl
- J1 pad 4: unconnected-(J1-Pin_4-Pad4) -> /top/sd_vl
- J2 pad 1: unconnected-(J2-Pin_1-Pad1) -> GND
- J2 pad 2: unconnected-(J2-Pin_2-Pad2) -> /top/3.3v
- J2 pad 3: unconnected-(J2-Pin_3-Pad3) -> /top/sc_vl
- J2 pad 4: unconnected-(J2-Pin_4-Pad4) -> /top/sd_vl
- J3 pad 1: unconnected-(J3-Pin_1-Pad1) -> GND
- J3 pad 2: unconnected-(J3-Pin_2-Pad2) -> /top/3.3v
- J3 pad 3: unconnected-(J3-Pin_3-Pad3) -> /top/sc_vl
- J3 pad 4: unconnected-(J3-Pin_4-Pad4) -> /top/sd_vl
- J4 pad 1: /sensorC/3.3v -> GND
- J4 pad 2: GND -> /sensorC/3.3v
- J4 pad 3: /sensorC/sd_vl -> /sensorC/sc_vl
- J4 pad 4: /sensorC/sc_vl -> /sensorC/sd_vl
- U1 pad 1: GND -> Net-(U1-SDO/SA0)
- U1 pad 12: /top/1.8v -> /back/3.3v
- U1 pad 13: /top/scimu -> /back/scimu
- U1 pad 14: /top/sdimu -> /back/sdimu
- U1 pad 5: /top/1.8v -> /back/3.3v
- U1 pad 8: /top/1.8v -> /back/3.3v
- U3 pad 13: /top/sdimu -> unconnected-(U3-SD4-Pad13)
- U3 pad 14: /top/scimu -> unconnected-(U3-SC4-Pad14)
- U3 pad 2: /top/1.8v -> Net-(U3-A0)
- U4 pad 1: unconnected-(U4-V_{DD(A)}-Pad1) -> /back/3.3v
- U4 pad 10: unconnected-(U4-V_{DD(B)}-Pad10) -> /back/3.3v
- U4 pad 2: unconnected-(U4-SDA-Pad2) -> /back/sdimu
- U4 pad 4: unconnected-(U4-SCL-Pad4) -> /back/scimu
- U5 pad 1: /sensorC/3.3v -> GND
- U5 pad 2: GND -> Net-(U5-SW)
- U5 pad 3: /sensorC/3.3v -> /back/3.3v
- U5 pad 4: unconnected-(U5-BYP/ADJ-Pad4) -> GND
- U5 pad 5: /sensorC/1.8v -> /back/bat+
Routing:
- net /sensorC/1.8v: track 0.00 -> 40.0 mm
- net /sensorC/3.3v: track 0.00 -> 18.6 mm
- net GND: track 0.00 -> 15.7 mm, vias 0 -> 15
- net /sensorC/sd_vl: track 0.00 -> 9.66 mm
- net /sensorC/sc_vl: track 0.00 -> 8.58 mm
- net /top/1.8v: track 8.21 -> 0.00 mm
- net Net-(U2-NCS): track 0.00 -> 4.88 mm
- net Net-(U2-INT): track 0.00 -> 4.52 mm
- net Net-(U2-SPI_I2C_N): track 0.00 -> 2.70 mm
- net Net-(U2-SYNC): track 0.00 -> 2.70 mm
- net Net-(U2-LPN): track 0.00 -> 2.68 mm
- added copper zone on F.Cu, net GND
Other:
- board size 189.2 x 82.2 mm -> 189.1 x 78.7 mm

Commit message: layout front top
Parts:
- removed C1: 100n, Capacitor_SMD:C_0603_1608Metric
- removed NT0: NetTie_3, Jumper:SolderJumper-3_P1.3mm_Bridged12_RoundedPad1.0x1.5mm
- added REF**: MountingHole_2.2mm_M2_DIN965, MountingHole:MountingHole_2.2mm_M2_DIN965, F.Cu at (64.9, 39.0)
- added REF**: MountingHole_2.2mm_M2_DIN965, MountingHole:MountingHole_2.2mm_M2_DIN965, F.Cu at (70.4, 48.4)
- J2: moved to B.Cu
- moved NT1 8.02 mm to (74.4, 44.6), turned to 90 degrees
- moved U3 7.27 mm to (80.0, 43.2), turned to 180 degrees
- moved C5 5.79 mm to (73.9, 41.5), turned to 180 degrees
- moved R7 0.80 mm to (80.3, 102.6)
- moved R6 0.76 mm to (80.3, 100.6)
- moved C3 0.57 mm to (77.2, 101.9)
- moved R4 0.36 mm to (74.9, 101.9)
- turned J2 to -90 degrees
Connections:
- J1 pad 1: GND -> /top/1.8v
- J1 pad 2: /top/3.3v -> /top/sd1
- J1 pad 3: /top/sc_vl -> /top/sc1
- J1 pad 4: /top/sd_vl -> /top/3.3v
- J1 pad 5: /top/1.8v -> GND
- J2 pad 1: GND -> /top/1.8v
- J2 pad 2: /top/3.3v -> /top/sd2
- J2 pad 3: /top/sc_vl -> /top/sc2
- J2 pad 4: /top/sd_vl -> /top/3.3v
- J2 pad 5: /top/1.8v -> GND
- J3 pad 1: GND -> /top/1.8v
- J3 pad 2: /top/3.3v -> /top/sd3
- J3 pad 3: /top/sc_vl -> /top/sc3
- J3 pad 4: /top/sd_vl -> /top/3.3v
- J3 pad 5: /top/1.8v -> GND
- J5 pad 1: unconnected-(J5-Pin_1-Pad1) -> /top/1.8v
- J5 pad 2: unconnected-(J5-Pin_2-Pad2) -> /top/scl
- J5 pad 3: unconnected-(J5-Pin_3-Pad3) -> /top/sda
- J5 pad 4: unconnected-(J5-Pin_4-Pad4) -> /top/3.3v
- J5 pad 5: unconnected-(J5-Pin_5-Pad5) -> GND
- J5 pad 6: unconnected-(J5-Pin_6-Pad6) -> GND
- U3 pad 10: /top/sd3 -> unconnected-(U3-SD3-Pad10)
- U3 pad 11: /top/sc3 -> unconnected-(U3-SC3-Pad11)
- U3 pad 13: unconnected-(U3-SD4-Pad13) -> /top/sd3
- U3 pad 14: unconnected-(U3-SC4-Pad14) -> /top/sc3
- U3 pad 2: Net-(U3-A0) -> /top/1.8v
Routing:
- net /top/1.8v: track 0.00 -> 96.3 mm, vias 0 -> 1
- net /top/3.3v: track 0.00 -> 59.6 mm, vias 0 -> 1
- net /top/sd3: track 0.00 -> 17.7 mm, vias 0 -> 2
- net /top/sc3: track 0.00 -> 16.6 mm, vias 0 -> 2
- net /top/sc1: track 0.00 -> 13.8 mm, vias 0 -> 2
- net /top/sda: track 0.00 -> 13.4 mm
- net GND: track 15.7 -> 28.5 mm, vias 15 -> 28
- net /top/sd1: track 0.00 -> 11.6 mm, vias 0 -> 2
- net /top/scl: track 0.00 -> 10.8 mm
- net /top/sd2: track 0.00 -> 10.6 mm, vias 0 -> 1
- net /top/sc2: track 0.00 -> 9.18 mm, vias 0 -> 1
- net Net-(U3-A1): track 0.00 -> 2.86 mm
- net /sensorC/1.8v: track 40.0 -> 41.4 mm
- net /sensorC/sc_vl: track 8.58 -> 9.83 mm
- net /sensorC/sd_vl: track 9.66 -> 10.3 mm
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Other:
- board text added: "1.8"
- board text added: "3.3"
- board text added: "gnd"
- board text added: "scl"
- board text added: "sda"

Commit message: push changes
Parts:
- added J7: Conn_01x08_Pin, Library:JST_XH_B8B-XH-AM_1x08_P2.50mm_Vertical, F.Cu at (235.7, 95.2)
- added REF**: MountingHole_2.2mm_M2_DIN965, MountingHole:MountingHole_2.2mm_M2_DIN965, F.Cu at (237.9, 81.9)
- added REF**: MountingHole_2.2mm_M2_DIN965, MountingHole:MountingHole_2.2mm_M2_DIN965, F.Cu at (200.9, 94.7)
- C12: footprint Capacitor_SMD:C_0402_1005Metric -> Capacitor_SMD:C_0603_1608Metric
- L1: footprint Inductor_SMD:L_Vishay_IHLP-3232 -> Library:WE-XHMI_4020
- R7: value R -> 2k
- moved C6 15.0 mm to (221.7, 85.1), turned to 180 degrees
- moved L1 13.4 mm to (199.0, 85.2)
- moved U4 12.2 mm to (231.9, 87.4), turned to -90 degrees
- moved C11 11.7 mm to (235.8, 87.9)
- moved C10 11.0 mm to (235.8, 86.1)
- moved C7 10.00 mm to (221.7, 82.5), turned to 180 degrees
- moved NT3 9.35 mm to (229.2, 81.3), turned to 180 degrees
- moved C14 8.33 mm to (210.9, 91.3), turned to 90 degrees
- moved C12 7.85 mm to (194.9, 90.6), turned to -90 degrees
- moved U5 6.88 mm to (194.3, 87.0)
- moved U1 6.17 mm to (225.2, 83.6), turned to -90 degrees
- moved L2 5.26 mm to (209.9, 94.7)
- moved R11 5.06 mm to (207.9, 88.9)
- moved C13 4.98 mm to (205.2, 92.1), turned to 90 degrees
- moved U6 4.95 mm to (207.9, 92.1)
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Connections:
- C12 pad 1: Net-(U5-MODE/S-CONF) -> Net-(U5-SS/TR)
- J6 pad 2: /back/3.3v -> /back/scimu
- J6 pad 3: GND -> /back/sdimu
- J6 pad 4: GND -> /back/3.3v
- J6 pad 5: /back/scimu -> GND
- J6 pad 6: /back/sdimu -> GND
- R8 pad 1: Net-(U5-SS/TR) -> Net-(U5-MODE/S-CONF)
- U4 pad 6: unconnected-(U4-DSCLM-Pad6) -> Net-(J7-Pin_4)
- U4 pad 7: unconnected-(U4-DSCLP-Pad7) -> Net-(J7-Pin_3)
- U4 pad 8: unconnected-(U4-DSDAP-Pad8) -> Net-(J7-Pin_2)
- U4 pad 9: unconnected-(U4-DSDAM-Pad9) -> Net-(J7-Pin_1)
Routing:
- net /back/3.3v: track 0.00 -> 107.4 mm
- net /back/bat+: track 0.00 -> 44.1 mm
- net /back/sdimu: track 0.00 -> 37.9 mm
- net /back/1.8v: track 0.00 -> 32.0 mm, vias 0 -> 3
- net /back/scimu: track 0.00 -> 31.3 mm
- net GND: track 28.5 -> 56.8 mm, vias 28 -> 95
- net Net-(J7-Pin_1): track 0.00 -> 7.10 mm
- net Net-(J7-Pin_4): track 0.00 -> 6.84 mm
- net Net-(J7-Pin_2): track 0.00 -> 6.27 mm
- net Net-(J7-Pin_3): track 0.00 -> 6.01 mm
- net Net-(U6-FB): track 0.00 -> 4.63 mm
- net Net-(U1-SDO/SA0): track 0.00 -> 4.27 mm
- net Net-(U5-FB/VSET): track 0.00 -> 3.42 mm
- net Net-(U5-MODE/S-CONF): track 0.00 -> 2.40 mm
- net Net-(U5-SS/TR): track 0.00 -> 2.12 mm
- added copper zone on F.Cu, net /back/1.8v
- added copper zone on F.Cu, net /back/3.3v
- added copper zone on F.Cu, net Net-(U5-SW)
- added copper zone on F.Cu, net Net-(U6-SW)
Other:
- outline, holes or cut-outs redrawn
